File: hardware/fmu-v2.kicad_sch (KiCad schematic)
At the start: 0 parts

Commit message: Take the carrier from schematic to a DRC-clean board; fix a dangling-net defect
Exporting the carrier as a standalone board netlist exposed a real design
defect: 28 of its nets terminated on a single pin. As a child sheet of
jfox-tmr that reads fine - the net continues into the FMU sheet - but a
pass-through carrier is a path, and half a path is not one. Each board had a
single power connector with nowhere for the power to go.

Redesigned so every signal enters on one connector and leaves on another:
brick power in (J4-J6) -> module J601 out (J7-J9), CAN to the modules
(J1-J3) daisy-chained. Nine connectors, twelve nets, zero single-pin nets.

Two things are deliberately no longer on this board. The servo/PWM breakout
is gone because how three boards' motor commands arbitrate into one output
is still unresolved - TmrVoter is not wired into motor_task - and copper is
the wrong place to record a guess; each module's J901 cables straight to its
ESCs meanwhile. The safety switch is gone because J702's SAFETY lands on
U801.PB5, the IO co-processor this firmware never runs, and neither J405 nor
J601 carries a pin to route it through, so it would have been decorative.

The carrier is now its own KiCad project. It has to be: the three FMU
modules are separately manufactured hardware, and a shared project would
make a board netlist try to place 421 module components on the carrier.

Board work:

- All nine connectors carry real footprints - Hirose DF13 vertical parts
  matching what the modules actually use.
- tools/gen_carrier_pcb.py writes an 80x60 mm two-layer outline with four M3
  holes on a 30.000 x 30.000 mm pattern. That pattern is read from the
  module's own PX4FMUv2.4.5.brd via `kicad-cli pcb import` - board import
  exists on the CLI even though schematic import does not - so a stacked
  module lines up rather than nearly lining up.
- Verified: DRC 0 violations, 0 unconnected. Gerbers, drill and job file all
  export; the drill file contains exactly four 3.2 mm N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
Changed lines of the file:
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@@
 (kicad_sch (version 20230819) (generator eeschema)
   (paper "A3")
-  (text "PX4FMUv2.4.5 - PLACEHOLDER.\\nReplace this sheet's contents with the real board via\\nFile > Import > Non-KiCad Schematic on\\nhardware/vendor/PX4FMUv2.4.5.sch (Eagle 7.1.0, 421 parts, 12 sheets),\\nthen attach the hierarchical labels below to the matching connectors:\\n  CAN_H/CAN_L -> J405 pins 2/3   VDD_5V_BRICK -> J601 pins 1/2\\n  BATT_V_SENS -> J601 pin 4      BATT_I_SENS  -> J601 pin 3\\n  SAFETY      -> J702 pin 3      FMU_CH1..6   -> J901 (via U901)\\nThis sheet is instantiated three times; edit it once." (at 25.4 25.4 0)
+  (text "PX4FMUv2.4.5 - PLACEHOLDER.\\nReplace this sheet's contents with the real board via\\nFile > Import > Non-KiCad Schematic on\\nhardware/vendor/PX4FMUv2.4.5.sch (Eagle 7.1.0, 421 parts, 12 sheets),\\nthen attach the hierarchical labels below to the matching connectors:\\n  CAN_H/CAN_L -> J405 pins 2/3   VDD_5V_BRICK -> J601 pins 1/2\\n  BATT_V_SENS -> J601 pin 4      BATT_I_SENS  -> J601 pin 3\\n  SAFETY      -> J702 pin 3\\nThis sheet is instantiated three times; edit it once." (at 25.4 25.4 0)
     (effects (font (size 1.27 1.27)) (justify left top))
   )
@@
     (effects (font (size 1.27 1.27)) (justify left))
   )
-  (hierarchical_label "FMU_CH1" (shape output) (at 50.8 91.44 0)
-    (effects (font (size 1.27 1.27)) (justify left))
-  )
-  (hierarchical_label "FMU_CH2" (shape output) (at 50.8 96.52 0)
-    (effects (font (size 1.27 1.27)) (justify left))
-  )
-  (hierarchical_label "FMU_CH3" (shape output) (at 50.8 101.6 0)
-    (effects (font (size 1.27 1.27)) (justify left))
-  )
-  (hierarchical_label "FMU_CH4" (shape output) (at 50.8 106.67999999999999 0)
-    (effects (font (size 1.27 1.27)) (justify left))
-  )
-  (hierarchical_label "FMU_CH5" (shape output) (at 50.8 111.75999999999999 0)
-    (effects (font (size 1.27 1.27)) (justify left))
-  )
-  (hierarchical_label "FMU_CH6" (shape output) (at 50.8 116.83999999999999 0)
-    (effects (font (size 1.27 1.27)) (justify left))
-  )
