File: hardware/fmu-v2/PX4FMUv2.4.5_11.kicad_sch (KiCad schematic)
At the start: 32 parts, among them J601 DF13C-6P-1.25V, U1101 LTC4417, U1102 NTHD4102PT1G, U1103 NTHD4102PT1G, U1104 NTHD4102PT1G

Commit message: Specify JFOX-FMU v1: STM32H753, 1 MB RAM, three IMUs per board
A ground-up replacement for the PX4FMUv2.4.5 modules, with that board as a
guideline only - its proven ideas kept, its limitations not. Specification
only; no schematic captured.

STM32H753IIT6, LQFP176: Cortex-M7 at 480 MHz, 1 MB RAM against the current
256 KB, and a hardware crypto block that the planned JFOXLink datalink can
use. LQFP rather than the BGA the same die also ships in, so hand assembly
stays possible. The pin structure is read from KiCad's own STM32H753IITx
symbol - 14x VDD, 2x VCAP, separate VDD33_USB, PDR_ON, 140 GPIO - not
recalled.

Sensors follow what Pixhawk FMUv6X actually ships, read from PX4's own
rc.board_sensors and spi.cpp: three IMUs from two vendors, each on its own
SPI bus with its own power-enable GPIO. The separate buses are the point -
one sensor hanging its bus, or needing a power cycle to recover, must not
take the other two with it. BMI088 (Bosch) + ICM-42688-P + ICM-45686 (TDK),
two barometers from two vendors, BMM150 internal magnetometer.

Recorded honestly rather than glossed: two of the three IMUs are TDK parts,
so a TDK-wide errata is not fully covered. FMUv6X makes the same compromise.
An ADI ADIS16470 in place of one buys genuine three-vendor diversity at
several times the cost, and is left as an open question.

The IO co-processor is dropped. This project's firmware has never run code on
it, which is exactly why the safety switch does nothing today - J702 lands on
U801.PB5, in a domain the FMU never initialises. The cost is that no
independent processor holds outputs safe if the FMU hangs; the watchdog and
board-level voting cover it, but that is a real difference from PX4 practice
and the spec says to argue it in the safety case rather than assume it away.

Two long-standing defects are designed out. CAN termination goes behind a
jumper, so the middle module of a three-board chain no longer needs R409
physically desoldered. And a 16 MHz crystal divides exact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
Parts:
- renumbered C1101 to C1101A1, C1102 to C1102A1, C1103 to C1103A1, C1104 to C1104A1, C1105 to C1105A1, C1106 to C1106A1, C1107 to C1107A1, C1108 to C1108A1, C1109 to C1109A1, C1110 to C1110A1, J601 to J601A1, L1101 to L1101A1, L1102 to L1102A1, R1101 to R1101A1, R1102 to R1102A1, R1103 to R1103A1, R1104 to R1104A1, R1105 to R1105A1, R1106 to R1106A1, R1107 to R1107A1, R1109 to R1109A1, R1110 to R1110A1, R1111 to R1111A1, R1112 to R1112A1, R1113 to R1113A1, R1114 to R1114A1, R1115 to R1115A1, RN1101 to RN1101A1, U1101 to U1101A1, U1102 to U1102A1, U1103 to U1103A1, U1104 to U1104A1
