File: hardware/fmu-v2/PX4FMUv2.4.5_12.kicad_sch (KiCad schematic)
At the start: 33 parts, among them M3_MOUNT1101 MOUNT-HOLE3.1MM, M3_MOUNT1102 MOUNT-HOLE3.1MM, M3_MOUNT1103 MOUNT-HOLE3.1MM, M3_MOUNT1104 MOUNT-HOLE3.1MM

Commit message: Specify JFOX-FMU v1: STM32H753, 1 MB RAM, three IMUs per board
A ground-up replacement for the PX4FMUv2.4.5 modules, with that board as a
guideline only - its proven ideas kept, its limitations not. Specification
only; no schematic captured.

STM32H753IIT6, LQFP176: Cortex-M7 at 480 MHz, 1 MB RAM against the current
256 KB, and a hardware crypto block that the planned JFOXLink datalink can
use. LQFP rather than the BGA the same die also ships in, so hand assembly
stays possible. The pin structure is read from KiCad's own STM32H753IITx
symbol - 14x VDD, 2x VCAP, separate VDD33_USB, PDR_ON, 140 GPIO - not
recalled.

Sensors follow what Pixhawk FMUv6X actually ships, read from PX4's own
rc.board_sensors and spi.cpp: three IMUs from two vendors, each on its own
SPI bus with its own power-enable GPIO. The separate buses are the point -
one sensor hanging its bus, or needing a power cycle to recover, must not
take the other two with it. BMI088 (Bosch) + ICM-42688-P + ICM-45686 (TDK),
two barometers from two vendors, BMM150 internal magnetometer.

Recorded honestly rather than glossed: two of the three IMUs are TDK parts,
so a TDK-wide errata is not fully covered. FMUv6X makes the same compromise.
An ADI ADIS16470 in place of one buys genuine three-vendor diversity at
several times the cost, and is left as an open question.

The IO co-processor is dropped. This project's firmware has never run code on
it, which is exactly why the safety switch does nothing today - J702 lands on
U801.PB5, in a domain the FMU never initialises. The cost is that no
independent processor holds outputs safe if the FMU hangs; the watchdog and
board-level voting cover it, but that is a real difference from PX4 practice
and the spec says to argue it in the safety case rather than assume it away.

Two long-standing defects are designed out. CAN termination goes behind a
jumper, so the middle module of a three-board chain no longer needs R409
physically desoldered. And a 16 MHz crystal divides exact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
Parts:
- renumbered !VBUS_VALID0 to !VBUS_VALID0A1, !VDD_BRICK_VALID0 to !VDD_BRICK_VALID0A1, !VDD_SERVO_VALID0 to !VDD_SERVO_VALID0A1, ADC_PR0 to ADC_PR0A1, CAN_H0 to CAN_H0A1, CAN_L0 to CAN_L0A1, FMU-BOOT1101 to FMU-BOOT1101A1, GND.0 to GND.0A1, GND0 to GND0A1, IO-BOOT1101 to IO-BOOT1101A1, JP1 to JP1A1, JP2 to JP2A1, M3_MOUNT1101 to M3_MOUNT1101A1, M3_MOUNT1102 to M3_MOUNT1102A1, M3_MOUNT1103 to M3_MOUNT1103A1, M3_MOUNT1104 to M3_MOUNT1104A1, OSHW_LOGO0 to OSHW_LOGO0A1, S1RX0 to S1RX0A1, S1TX0 to S1TX0A1, S2RX0 to S2RX0A1, S2TX0 to S2TX0A1, S3RX0 to S3RX0A1, S3TX0 to S3TX0A1, S4RX0 to S4RX0A1, S4TX0 to S4TX0A1, S5_RX0 to S5_RX0A1, S5_TX0 to S5_TX0A1, VBUS0 to VBUS0A1, VDDA_3V1101 to VDDA_3V1101A1, VDD_3V1101 to VDD_3V1101A1, VDD_5V_BRICK0 to VDD_5V_BRICK0A1, VDD_5V_IN0 to VDD_5V_IN0A1, VDD_SERVO0 to VDD_SERVO0A1
