File: hardware/fmu-v2/PX4FMUv2.4.5_2.kicad_sch (KiCad schematic)
At the start: 30 parts, among them J201 DF13C-6P-1.25V, J202 DF13C-6P-1.25V, J203 DF13C-6P-1.25V, J204 DF13C-6P-1.25V, U201 TXS0108QFN20, U202 TXS0108QFN20

Commit message: Specify JFOX-FMU v1: STM32H753, 1 MB RAM, three IMUs per board
A ground-up replacement for the PX4FMUv2.4.5 modules, with that board as a
guideline only - its proven ideas kept, its limitations not. Specification
only; no schematic captured.

STM32H753IIT6, LQFP176: Cortex-M7 at 480 MHz, 1 MB RAM against the current
256 KB, and a hardware crypto block that the planned JFOXLink datalink can
use. LQFP rather than the BGA the same die also ships in, so hand assembly
stays possible. The pin structure is read from KiCad's own STM32H753IITx
symbol - 14x VDD, 2x VCAP, separate VDD33_USB, PDR_ON, 140 GPIO - not
recalled.

Sensors follow what Pixhawk FMUv6X actually ships, read from PX4's own
rc.board_sensors and spi.cpp: three IMUs from two vendors, each on its own
SPI bus with its own power-enable GPIO. The separate buses are the point -
one sensor hanging its bus, or needing a power cycle to recover, must not
take the other two with it. BMI088 (Bosch) + ICM-42688-P + ICM-45686 (TDK),
two barometers from two vendors, BMM150 internal magnetometer.

Recorded honestly rather than glossed: two of the three IMUs are TDK parts,
so a TDK-wide errata is not fully covered. FMUv6X makes the same compromise.
An ADI ADIS16470 in place of one buys genuine three-vendor diversity at
several times the cost, and is left as an open question.

The IO co-processor is dropped. This project's firmware has never run code on
it, which is exactly why the safety switch does nothing today - J702 lands on
U801.PB5, in a domain the FMU never initialises. The cost is that no
independent processor holds outputs safe if the FMU hangs; the watchdog and
board-level voting cover it, but that is a real difference from PX4 practice
and the spec says to argue it in the safety case rather than assume it away.

Two long-standing defects are designed out. CAN termination goes behind a
jumper, so the middle module of a three-board chain no longer needs R409
physically desoldered. And a 16 MHz crystal divides exact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
Parts:
- renumbered C201 to C201A1, C202 to C202A1, D201 to D201A1, D202 to D202A1, D203 to D203A1, J201 to J201A1, J202 to J202A1, J203 to J203A1, J204 to J204A1, L201 to L201A1, L202 to L202A1, L203 to L203A1, R201 to R201A1, R202 to R202A1, R203 to R203A1, R204 to R204A1, R205 to R205A1, R206 to R206A1, R207 to R207A1, R208 to R208A1, R209 to R209A1, R210 to R210A1, R211 to R211A1, R212 to R212A1, R213 to R213A1, R214 to R214A1, R215 to R215A1, R216 to R216A1, U201 to U201A1, U202 to U202A1
