File: hardware/fmu-v2/PX4FMUv2.4.5_3.kicad_sch (KiCad schematic)
At the start: 12 parts, among them J301 47346-0001, J302 DF13C-4P-1.25V, U301 2908-05WB-MG, U302 NUF2042XV6

Commit message: Specify JFOX-FMU v1: STM32H753, 1 MB RAM, three IMUs per board
A ground-up replacement for the PX4FMUv2.4.5 modules, with that board as a
guideline only - its proven ideas kept, its limitations not. Specification
only; no schematic captured.

STM32H753IIT6, LQFP176: Cortex-M7 at 480 MHz, 1 MB RAM against the current
256 KB, and a hardware crypto block that the planned JFOXLink datalink can
use. LQFP rather than the BGA the same die also ships in, so hand assembly
stays possible. The pin structure is read from KiCad's own STM32H753IITx
symbol - 14x VDD, 2x VCAP, separate VDD33_USB, PDR_ON, 140 GPIO - not
recalled.

Sensors follow what Pixhawk FMUv6X actually ships, read from PX4's own
rc.board_sensors and spi.cpp: three IMUs from two vendors, each on its own
SPI bus with its own power-enable GPIO. The separate buses are the point -
one sensor hanging its bus, or needing a power cycle to recover, must not
take the other two with it. BMI088 (Bosch) + ICM-42688-P + ICM-45686 (TDK),
two barometers from two vendors, BMM150 internal magnetometer.

Recorded honestly rather than glossed: two of the three IMUs are TDK parts,
so a TDK-wide errata is not fully covered. FMUv6X makes the same compromise.
An ADI ADIS16470 in place of one buys genuine three-vendor diversity at
several times the cost, and is left as an open question.

The IO co-processor is dropped. This project's firmware has never run code on
it, which is exactly why the safety switch does nothing today - J702 lands on
U801.PB5, in a domain the FMU never initialises. The cost is that no
independent processor holds outputs safe if the FMU hangs; the watchdog and
board-level voting cover it, but that is a real difference from PX4 practice
and the spec says to argue it in the safety case rather than assume it away.

Two long-standing defects are designed out. CAN termination goes behind a
jumper, so the middle module of a three-board chain no longer needs R409
physically desoldered. And a 16 MHz crystal divides exact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
Parts:
- renumbered J301 to J301A1, J302 to J302A1, JX301 to JX301A1, R301 to R301A1, R302 to R302A1, R303 to R303A1, R304 to R304A1, R305 to R305A1, R306 to R306A1, R307 to R307A1, U301 to U301A1, U302 to U302A1
