File: hardware/fmu-v2/PX4FMUv2.4.5_5.kicad_sch (KiCad schematic)
At the start: 21 parts, among them U501 L3GD20, U502 L3GD20H, U504 LSM303D, U505 MPU-6000, U506 MS5611-01BA, X503 0512811094

Commit message: Specify JFOX-FMU v1: STM32H753, 1 MB RAM, three IMUs per board
A ground-up replacement for the PX4FMUv2.4.5 modules, with that board as a
guideline only - its proven ideas kept, its limitations not. Specification
only; no schematic captured.

STM32H753IIT6, LQFP176: Cortex-M7 at 480 MHz, 1 MB RAM against the current
256 KB, and a hardware crypto block that the planned JFOXLink datalink can
use. LQFP rather than the BGA the same die also ships in, so hand assembly
stays possible. The pin structure is read from KiCad's own STM32H753IITx
symbol - 14x VDD, 2x VCAP, separate VDD33_USB, PDR_ON, 140 GPIO - not
recalled.

Sensors follow what Pixhawk FMUv6X actually ships, read from PX4's own
rc.board_sensors and spi.cpp: three IMUs from two vendors, each on its own
SPI bus with its own power-enable GPIO. The separate buses are the point -
one sensor hanging its bus, or needing a power cycle to recover, must not
take the other two with it. BMI088 (Bosch) + ICM-42688-P + ICM-45686 (TDK),
two barometers from two vendors, BMM150 internal magnetometer.

Recorded honestly rather than glossed: two of the three IMUs are TDK parts,
so a TDK-wide errata is not fully covered. FMUv6X makes the same compromise.
An ADI ADIS16470 in place of one buys genuine three-vendor diversity at
several times the cost, and is left as an open question.

The IO co-processor is dropped. This project's firmware has never run code on
it, which is exactly why the safety switch does nothing today - J702 lands on
U801.PB5, in a domain the FMU never initialises. The cost is that no
independent processor holds outputs safe if the FMU hangs; the watchdog and
board-level voting cover it, but that is a real difference from PX4 practice
and the spec says to argue it in the safety case rather than assume it away.

Two long-standing defects are designed out. CAN termination goes behind a
jumper, so the middle module of a three-board chain no longer needs R409
physically desoldered. And a 16 MHz crystal divides exact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
Parts:
- renumbered C501 to C501A1, C502 to C502A1, C503 to C503A1, C504 to C504A1, C505 to C505A1, C506 to C506A1, C507 to C507A1, C508 to C508A1, C509 to C509A1, C510 to C510A1, C511 to C511A1, C512 to C512A1, C513 to C513A1, C514 to C514A1, C515 to C515A1, U501 to U501A1, U502 to U502A1, U504 to U504A1, U505 to U505A1, U506 to U506A1, X503 to X503A1
