File: hardware/fmu-v2/PX4FMUv2.4.5_6.kicad_sch (KiCad schematic)
At the start: 40 parts, among them Q601 MMBT3906SMDLT1, U101 STM32F4X7VX, U601 BQ24315, U602 BQ24315, U603 MIC5332

Commit message: Specify JFOX-FMU v1: STM32H753, 1 MB RAM, three IMUs per board
A ground-up replacement for the PX4FMUv2.4.5 modules, with that board as a
guideline only - its proven ideas kept, its limitations not. Specification
only; no schematic captured.

STM32H753IIT6, LQFP176: Cortex-M7 at 480 MHz, 1 MB RAM against the current
256 KB, and a hardware crypto block that the planned JFOXLink datalink can
use. LQFP rather than the BGA the same die also ships in, so hand assembly
stays possible. The pin structure is read from KiCad's own STM32H753IITx
symbol - 14x VDD, 2x VCAP, separate VDD33_USB, PDR_ON, 140 GPIO - not
recalled.

Sensors follow what Pixhawk FMUv6X actually ships, read from PX4's own
rc.board_sensors and spi.cpp: three IMUs from two vendors, each on its own
SPI bus with its own power-enable GPIO. The separate buses are the point -
one sensor hanging its bus, or needing a power cycle to recover, must not
take the other two with it. BMI088 (Bosch) + ICM-42688-P + ICM-45686 (TDK),
two barometers from two vendors, BMM150 internal magnetometer.

Recorded honestly rather than glossed: two of the three IMUs are TDK parts,
so a TDK-wide errata is not fully covered. FMUv6X makes the same compromise.
An ADI ADIS16470 in place of one buys genuine three-vendor diversity at
several times the cost, and is left as an open question.

The IO co-processor is dropped. This project's firmware has never run code on
it, which is exactly why the safety switch does nothing today - J702 lands on
U801.PB5, in a domain the FMU never initialises. The cost is that no
independent processor holds outputs safe if the FMU hangs; the watchdog and
board-level voting cover it, but that is a real difference from PX4 practice
and the spec says to argue it in the safety case rather than assume it away.

Two long-standing defects are designed out. CAN termination goes behind a
jumper, so the middle module of a three-board chain no longer needs R409
physically desoldered. And a 16 MHz crystal divides exact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
Parts:
- renumbered B601 to B601A1, C601 to C601A1, C602 to C602A1, C603 to C603A1, C604 to C604A1, C605 to C605A1, C606 to C606A1, C607 to C607A1, C608 to C608A1, C609 to C609A1, C610 to C610A1, C611 to C611A1, C612 to C612A1, C613 to C613A1, C614 to C614A1, C615 to C615A1, C616 to C616A1, C617 to C617A1, C618 to C618A1, D602 to D602A1, L603 to L603A1, Q601 to Q601A1, R602 to R602A1, R603 to R603A1, R604 to R604A1, R608 to R608A1, R609 to R609A1, R610 to R610A1, R611 to R611A1, R615 to R615A1, R616 to R616A1, R617 to R617A1, R620 to R620A1, R621 to R621A1, R635 to R635A1, S601 to S601A1, U101 to U101A1, U601 to U601A1, U602 to U602A1, U603 to U603A1
