File: hardware/fmu-v2/PX4FMUv2.4.5_7.kicad_sch (KiCad schematic)
At the start: 31 parts, among them J701 DF13C-2P-1.25V, J702 DF13C-3P-1.25V, U701 TCA62724FMG, U702 LT3469, U703 LRTB GFTG-T7AW-1+V7A7-29+R5T9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

Commit message: Specify JFOX-FMU v1: STM32H753, 1 MB RAM, three IMUs per board
A ground-up replacement for the PX4FMUv2.4.5 modules, with that board as a
guideline only - its proven ideas kept, its limitations not. Specification
only; no schematic captured.

STM32H753IIT6, LQFP176: Cortex-M7 at 480 MHz, 1 MB RAM against the current
256 KB, and a hardware crypto block that the planned JFOXLink datalink can
use. LQFP rather than the BGA the same die also ships in, so hand assembly
stays possible. The pin structure is read from KiCad's own STM32H753IITx
symbol - 14x VDD, 2x VCAP, separate VDD33_USB, PDR_ON, 140 GPIO - not
recalled.

Sensors follow what Pixhawk FMUv6X actually ships, read from PX4's own
rc.board_sensors and spi.cpp: three IMUs from two vendors, each on its own
SPI bus with its own power-enable GPIO. The separate buses are the point -
one sensor hanging its bus, or needing a power cycle to recover, must not
take the other two with it. BMI088 (Bosch) + ICM-42688-P + ICM-45686 (TDK),
two barometers from two vendors, BMM150 internal magnetometer.

Recorded honestly rather than glossed: two of the three IMUs are TDK parts,
so a TDK-wide errata is not fully covered. FMUv6X makes the same compromise.
An ADI ADIS16470 in place of one buys genuine three-vendor diversity at
several times the cost, and is left as an open question.

The IO co-processor is dropped. This project's firmware has never run code on
it, which is exactly why the safety switch does nothing today - J702 lands on
U801.PB5, in a domain the FMU never initialises. The cost is that no
independent processor holds outputs safe if the FMU hangs; the watchdog and
board-level voting cover it, but that is a real difference from PX4 practice
and the spec says to argue it in the safety case rather than assume it away.

Two long-standing defects are designed out. CAN termination goes behind a
jumper, so the middle module of a three-board chain no longer needs R409
physically desoldered. And a 16 MHz crystal divides exact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
Parts:
- renumbered C701 to C701A1, C702 to C702A1, C703 to C703A1, C704 to C704A1, D701 to D701A1, J701 to J701A1, J702 to J702A1, L701 to L701A1, LED701 to LED701A1, LED702 to LED702A1, LED703 to LED703A1, LED704 to LED704A1, LED705 to LED705A1, R701 to R701A1, R702 to R702A1, R703 to R703A1, R704 to R704A1, R705 to R705A1, R706 to R706A1, R707 to R707A1, R708 to R708A1, R709 to R709A1, R710 to R710A1, R711 to R711A1, R712 to R712A1, R713 to R713A1, R735 to R735A1, R736 to R736A1, U701 to U701A1, U702 to U702A1, U703 to U703A1
