File: hardware/fmu-v2/PX4FMUv2.4.5_9.kicad_sch (KiCad schematic)
At the start: 32 parts, among them J901 HEADER-3X163X16RA, U901 TXS0108QFN20, U902 TXS0108QFN20, U903 74LVC2G240

Commit message: Specify JFOX-FMU v1: STM32H753, 1 MB RAM, three IMUs per board
A ground-up replacement for the PX4FMUv2.4.5 modules, with that board as a
guideline only - its proven ideas kept, its limitations not. Specification
only; no schematic captured.

STM32H753IIT6, LQFP176: Cortex-M7 at 480 MHz, 1 MB RAM against the current
256 KB, and a hardware crypto block that the planned JFOXLink datalink can
use. LQFP rather than the BGA the same die also ships in, so hand assembly
stays possible. The pin structure is read from KiCad's own STM32H753IITx
symbol - 14x VDD, 2x VCAP, separate VDD33_USB, PDR_ON, 140 GPIO - not
recalled.

Sensors follow what Pixhawk FMUv6X actually ships, read from PX4's own
rc.board_sensors and spi.cpp: three IMUs from two vendors, each on its own
SPI bus with its own power-enable GPIO. The separate buses are the point -
one sensor hanging its bus, or needing a power cycle to recover, must not
take the other two with it. BMI088 (Bosch) + ICM-42688-P + ICM-45686 (TDK),
two barometers from two vendors, BMM150 internal magnetometer.

Recorded honestly rather than glossed: two of the three IMUs are TDK parts,
so a TDK-wide errata is not fully covered. FMUv6X makes the same compromise.
An ADI ADIS16470 in place of one buys genuine three-vendor diversity at
several times the cost, and is left as an open question.

The IO co-processor is dropped. This project's firmware has never run code on
it, which is exactly why the safety switch does nothing today - J702 lands on
U801.PB5, in a domain the FMU never initialises. The cost is that no
independent processor holds outputs safe if the FMU hangs; the watchdog and
board-level voting cover it, but that is a real difference from PX4 practice
and the spec says to argue it in the safety case rather than assume it away.

Two long-standing defects are designed out. CAN termination goes behind a
jumper, so the middle module of a three-board chain no longer needs R409
physically desoldered. And a 16 MHz crystal divides exact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
Parts:
- renumbered C901 to C901A1, C902 to C902A1, C903 to C903A1, D901 to D901A1, D902 to D902A1, D903 to D903A1, D904 to D904A1, J901 to J901A1, L901 to L901A1, R901 to R901A1, R902 to R902A1, R903 to R903A1, R904 to R904A1, R905 to R905A1, R906 to R906A1, R907 to R907A1, R908 to R908A1, R909 to R909A1, R910 to R910A1, R911 to R911A1, R912 to R912A1, R913 to R913A1, R914 to R914A1, R915 to R915A1, R916 to R916A1, R917 to R917A1, R918 to R918A1, R919 to R919A1, R922 to R922A1, U901 to U901A1, U902 to U902A1, U903 to U903A1
