File: hardware/jfox-fmu-v1/power.kicad_sch (KiCad schematic)
At the start: 7 parts, among them U20 LTC4417CGN, U21 TPS62132, U22 AP2112K-3.3, U23 AP22804AW5, U24 AP22804AW5, U25 AP22804AW5, U26 AP22804AW5

Commit message: Footprint every part, and verify each one exists
58 of 58 components now carry a footprint chosen against the package its
datasheet specifies, and check_fmu_footprints.py confirms every name resolves
to a file on disk.

Three of the names this design was carrying did not. The symbol library named
`Sensor_Motion:InvenSense_QFN-14_3x3mm_P0.5mm` and
`Sensor_Pressure:Bosch_LGA-10_2x2mm_P0.35mm`, neither of which is a footprint
in any installed library - both plausible, both fiction. The third was worse:
`Package_LGA:Bosch_LGA-14_3x2.5mm_P0.5mm` is real, matches the InvenSense
package on every word of its name, and is drawn for the BMI160 with 0.675 mm
pads where InvenSense wants 0.475 mm.

Notable choices, each traceable:
  LTC4417CGN  GN is the 16-lead narrow SSOP.
  TPS62132    RGT 3x3 VQFN. TI's land drawing (4222419/E) gives the exposed
              pad as 1.55 mm; KiCad's 1.6 mm variant is closest. Thermal-via
              variant, since the datasheet is explicit that the pad must be
              soldered and that dissipation limits output power.
  Bulk caps   4u7/10u/22u get an 0805, not the 0402 every other capacitor
              gets. Assigning one size to all of them produces a board that
              cannot be built from the BOM it ships with.
  L1          a generic 1210 land, and labelled as such - the 2.2 uH part is
              not chosen yet, since saturation current and DCR still have to
              be picked against the real 550 mA peak.

The checker was wrong on its first run, in a way worth recording because the
failure mode is self-concealing. It matched ref, value and footprint in one
regex with the footprint group optional, so a component with no footprint -
precisely what it exists to find - failed to match at all, dropped out of the
list, and the run reported "every component maps to a footprint" while the
count quietly fell by one. A check whose failure mode is to stop seeing the
failure is worse than no check. Now it splits into per-com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
Parts:
- U20: footprint (none) -> Package_SO:SSOP-16_3.9x4.9mm_P0.635mm
- U21: footprint (none) -> Package_DFN_QFN:VQFN-16-1EP_3x3mm_P0.5mm_EP1.6x1.6mm_ThermalVias
- U22, U23, U24, U25, U26: footprint (none) -> Package_TO_SOT_SMD:SOT-23-5
Changed lines of the file:
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@@
+		)
+		)
+		(property "Footprint" "Package_SO:SSOP-16_3.9x4.9mm_P0.635mm"
+			(at 64.77 109.22 0)
+			(hide yes)
+			(effects
+			(font
+				(size 1.27 1.27)
+			)
 		)
 		)
 		(instances
 			(project "jfox-fmu"
-				(path "/d1e8a681-6ee5-4e7f-b035-aebe49eafd3e"
+				(path "/d24bd7c9-075b-4474-9e8a-0d94278e4e1b"
 					(reference "U20")
 					(unit 1)
@@
 		)
 		)
+		(property "Footprint" "Package_DFN_QFN:VQFN-16-1EP_3x3mm_P0.5mm_EP1.6x1.6mm_ThermalVias"
+			(at 142.24 83.82 0)
+			(hide yes)
+			(effects
+			(font
+				(size 1.27 1.27)
+			)
+		)
+		)
 		(instances
 			(project "jfox-fmu"
-				(path "/d1e8a681-6ee5-4e7f-b035-aebe49eafd3e"
+				(path "/d24bd7c9-075b-4474-9e8a-0d94278e4e1b"
 					(reference "U21")
 					(unit 1)
@@
 		)
 		)
+		(property "Footprint" "Package_TO_SOT_SMD:SOT-23-5"
+			(at 142.24 139.7 0)
+			(hide yes)
+			(effects
+			(font
+				(size 1.27 1.27)
+			)
+		)
+		)
 		(instances
 			(project "jfox-fmu"
-				(path "/d1e8a681-6ee5-4e7f-b035-aebe49eafd3e"
+				(path "/d24bd7c9-075b-4474-9e8a-0d94278e4e1b"
 					(reference "U22")
 					(unit 1)
@@
 		)
 		)
+		(property "Footprint" "Package_TO_SOT_SMD:SOT-23-5"
+			(at 78.74 189.23 0)
+			(hide yes)
+			(effects
+			(font
+				(size 1.27 1.27)
+			)
+		)
+		)
 		(instances
 			(project "jfox-fmu"
-				(path "/d1e8a681-6ee5-4e7f-b035-aebe49eafd3e"
+				(path "/d24bd7c9-075b-4474-9e8a-0d94278e4e1b"
 					(reference "U23")
 					(unit 1)
@@
 		)
 		)
+		(property "Footprint" "Package_TO_SOT_SMD:SOT-23-5"
+			(at 157.48 189.23 0)
+			(hide yes)
+			(effects
+			(font
+				(size 1.27 1.27)
+			)
+		)
+		)
 		(instances
 			(project "jfox-fmu"
-				(path "/d1e8a681-6ee5-4e7f-b035-aebe49eafd3e"
+				(path "/d24bd7c9-075b-4474-9e8a-0d94278e4e1b"
 					(reference "U24")
 					(unit 1)
@@
 		)
 		)
+		(property "Footprint" "Package_TO_SOT_SMD:SOT-23-5"
+			(at 78.74 233.68 0)
+			(hide yes)
+			(effects
+			(font
+				(size 1.27 1.27)
+			)
+		)
+		)
 		(instances
 			(project "jfox-fmu"
-				(path "/d1e8a681-6ee5-4e7f-b035-aebe49eafd3e"
+				(path "/d24bd7c9-075b-4474-9e8a-0d94278e4e1b"
 					(reference "U25")
 					(unit 1)
@@
 		)
 		)
+		(property "Footprint" "Package_TO_SOT_SMD:SOT-23-5"
+			(at 157.48 233.68 0)
+			(hide yes)
+			(effects
+			(font
+				(size 1.27 1.27)
+			)
+		)
+		)
 		(instances
 			(project "jfox-fmu"
-				(path "/d1e8a681-6ee5-4e7f-b035-aebe49eafd3e"
+				(path "/d24bd7c9-075b-4474-9e8a-0d94278e4e1b"
 					(reference "U26")
 					(unit 1)
