File: hardware/jfox-fmu-v1/jfox-fmu.kicad_pcb (KiCad board)
At the start: 6 copper layers, 40 x 90 mm, 106 parts, among them J12 CAN1, J13 CAN2, J30 USB-C, J31 microSD, J40 CARD EDGE 2x30 P1.27 (no part), U1 ICM-42688-P, U10 STM32H753IIT6, U2 ICM-45686, U21 TPS62132, U22 AP2112K-3.3, U23 AP22804AW5, U24 AP22804AW5, U25 AP22804AW5, U26 AP22804AW5, U3 BMI088, U30 ISOW1044, U31 ISOW1044, U4 BMP388, U40 USBLC6-2SC6, U5 FM25V02A, U6 BMM150, U7 ICP-20100, X1 16MHz, X2 32.768kHz

Commit message: Provability: check the backplane, and fix the four defects that found
Nothing read JFOX-BASE-v1. Every checker in hardware/tools/ opened
jfox-fmu-v1/jfox-fmu.kicad_sch and only that, so no claim about the
backplane was provable - including the ones the requirements table recorded
as verified.

check_base_schematic.py now reads it: fused rails must reach a card socket,
the LTC4417 divider must produce the window it claims, that window must fit
every part downstream, and the feed-health outputs must reach a card AND be
driven. It failed on first run, which is the only reason to trust it.

What it found, in the order it found them:

  1. THE CARDS HAD NO POWER. The fuses put out A/B/C_FUSED and the card edge
     reads +5V_CARRIER. Both boards generated cleanly, both passed DRC, and
     the two halves were never connected to each other. The chain now
     terminates on the card rail past the shunt, not before it.

  2. THE FEEDS ARE NOT BATTERIES. VBAT_RH/VBAT_LH carry 5 V - the thresholds
     said so and the connectors are labelled PWR. Renamed PWR1_IN/PWR2_IN,
     output PWR_ORED. The name was the thing that was wrong.

  3. THE WINDOW PASSED MORE THAN A PART SURVIVES, and the binding part was
     not the one found by hand. The analysis flagged the AP2112K at 6.0 V
     against a 5.81 V threshold - 190 mV. The checker compared against every
     downstream part and found the ISOW1044 at 5.5 V: NEGATIVE 310 mV. A
     feed the controller reported as good would have destroyed the isolator.

     787k / 28k7 / 196k -> UV 4.50 V, OV 5.16 V
       ISOW1044  +338 mV      AP2112K  +838 mV

  4. THE ORING CONTROLLER'S OUTPUT WAS NEVER CONNECTED. Its pin map was
     written from the datasheet's block diagram, not the symbol: the pins
     are ~{VALID1..3} with overbars, VOUT not OUT, HYS not HYST, and there
     is no STAT pin at all. nets.get() returns None for an unknown key, so
     six pins were silently left unwired - VOUT among them. PWR_ORED was fed
     only by D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
Connections:
- J40 pad 55: BRICK_VALID -> PWR1_VALID
- J40 pad 57: SERVO_VALID -> PWR2_VALID
- J40 pad 58: USB_VALID -> unconnected-(J40-Pin_58-Pad58)
