File: hardware/jfox-base-v1/jfox-base.kicad_pcb (KiCad board)
At the start: 8 copper layers, 100 x 100 mm, 50 parts, among them J1 Mezz A, J2 Mezz B, J3 Mezz C, J50 PWR 1 RH, J51 PWR 2 LH, J52 DEBUG, J54 USB-C, J60 A CAN1, J61 A CAN2, J62 B CAN1, J63 B CAN2, J64 C CAN1, J65 C CAN2, J70 VEHICLE CAN, J80 ACT A, J81 ACT B, J82 ACT C, J90 GPS1 (A), J91 RC IN (B), J92 TELEM1 (A), J93 TELEM2 (C), U50 OPT1 TX, U51 OPT1 RX, U52 OPT2 TX, U53 OPT2 RX

Commit message: LTC4417 lands on the backplane, replacing the diode OR
It left the FCU when the power tree moved and never arrived here - the
backplane has been ORing its two airframe feeds with a pair of Schottkys,
which works and throws away the two things the part was chosen for:

  * Priority. A diode OR takes whichever feed is momentarily higher, so two
    supplies sitting 100 mV apart make the board chatter between them. The
    LTC4417 holds its selection until that source leaves its window.
  * A window. Under- and over-voltage per input, so a feed that has drifted
    out of spec is rejected rather than used because it is the higher of two
    bad ones.

It also drops ~0.4 V across a 5 V rail that the PMOS pass devices do not.

Two inputs, not three. V3 is tied to ground and its pass FET omitted, which
is how the datasheet says to leave an input out; inventing a third feed to
fill it would be worse. D50/D51 stay as reverse-polarity protection.

Three faults surfaced while wiring it, none of them the ORing:

  * The actuator headers still asked each channel for VDD_SERVO. That rail
    left the card's pinout when the power tree moved - servo power now runs
    from the backplane straight to the actuators and never passes through a
    card, which is the right way round. Three nets had nothing driving them.
  * EN was tied to +3V3, a rail the backplane does not have. It regulates
    nothing; the cards do. Now tied to the primary feed, so the part is
    enabled whenever there is power at all.
  * The expansion header overflowed. Its guard reported "25 spare signals
    will not fit a 20-pin header - widen it rather than dropping the
    overflow silently", which is exactly what it was written to catch. 2x15.

The far-face hole check earned itself again: a threshold divider placed on
the back landed under a card socket's through-holes. Bands on the back face
have to thread between sockets at y 20..27, 46..53 and 72..79.

  FCU        DRC 0 blocking, 105 parts, all checks pa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
Parts:
- removed MH1, MH2, MH3, MH4: M3, MountingHole_3.2mm_M3
- added C70: 100n, C_0402_1005Metric, B.Cu at (66.3, 96.6)
- added C71: 100n, C_0402_1005Metric, B.Cu at (68.7, 96.6)
- added J100: EXP A, PinHeader_2x10_P1.27mm_Vertical_SMD, B.Cu at (60.3, 66.8)
- added J101: EXP B, PinHeader_2x10_P1.27mm_Vertical_SMD, B.Cu at (70.1, 66.8)
- added J102: EXP C, PinHeader_2x10_P1.27mm_Vertical_SMD, B.Cu at (79.8, 66.8)
- added Q1A: PMOS, SOT-23, F.Cu at (81.6, 87.7)
- added Q1B: PMOS, SOT-23, F.Cu at (86.3, 87.7)
- added Q2A: PMOS, SOT-23, F.Cu at (91.0, 87.7)
- added Q2B: PMOS, SOT-23, F.Cu at (95.6, 87.7)
- added R70: 787k, R_0402_1005Metric, B.Cu at (99.3, 86.5)
- added R71: 49k9, R_0402_1005Metric, B.Cu at (101.6, 86.5)
- added R72: 174k, R_0402_1005Metric, B.Cu at (56.9, 96.6)
- added R73: 787k, R_0402_1005Metric, B.Cu at (59.3, 96.6)
- added R74: 49k9, R_0402_1005Metric, B.Cu at (61.6, 96.6)
- added R75: 174k, R_0402_1005Metric, B.Cu at (64.0, 96.6)
- added U20: LTC4417CGN, SSOP-24_3.9x8.7mm_P0.635mm, F.Cu at (59.5, 90.7)
- J1, J2, J3: footprint Samtec_MECF-30-01-NP-L-DV_2x30_P1.27mm_Socket_Horizontal -> Samtec_MECF-30-01-L-DV_2x30_P1.27mm_Polarized_Socket_Horizontal
- moved D50 39.3 mm to (67.6, 87.8)
- moved D51 32.8 mm to (75.4, 87.8)
- moved C50 25.7 mm to (86.2, 60.5)
- moved C51 25.0 mm to (88.6, 60.5)
- moved R41 12.0 mm to (106.3, 89.7)
- moved R40 10.8 mm to (103.9, 89.7)
- moved J65 2.00 mm to (107.7, 85.2)
- moved J64 1.60 mm to (107.7, 78.0)
- moved J63 1.20 mm to (107.7, 70.8)
- moved R61 1.17 mm to (52.5, 75.5)
- moved R62 1.17 mm to (52.5, 101.5)
- moved R60 1.17 mm to (52.5, 49.5)
- moved J62 0.80 mm to (107.7, 63.6)
- moved R2 0.57 mm to (50.1, 75.5)
- moved R3 0.57 mm to (50.1, 101.5)
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Connections:
- J1 pad 2: A_VDD_BRICK -> A_SWDIO
- J1 pad 3: A_VDD_BRICK -> A_SWCLK
- J1 pad 5: A_VDD_SERVO -> A_NRST
- J1 pad 54: unconnected-(J1-Pin_54-Pad54) -> A_USART1_RX
- J1 pad 55: unconnected-(J1-Pin_55-Pad55) -> A_BRICK_VALID
- J1 pad 57: unconnected-(J1-Pin_57-Pad57) -> A_SERVO_VALID
- J1 pad 58: unconnected-(J1-Pin_58-Pad58) -> A_USB_VALID
- J1 pad 59: GND -> A_TIM4_CH4
- J1 pad 6: A_VDD_SERVO -> A_USART1_TX
- J2 pad 2: B_VDD_BRICK -> B_SWDIO
- J2 pad 3: B_VDD_BRICK -> B_SWCLK
- J2 pad 5: B_VDD_SERVO -> B_NRST
- J2 pad 54: unconnected-(J2-Pin_54-Pad54) -> B_USART1_RX
- J2 pad 55: unconnected-(J2-Pin_55-Pad55) -> B_BRICK_VALID
- J2 pad 57: unconnected-(J2-Pin_57-Pad57) -> B_SERVO_VALID
- J2 pad 58: unconnected-(J2-Pin_58-Pad58) -> B_USB_VALID
- J2 pad 59: GND -> B_TIM4_CH4
- J2 pad 6: B_VDD_SERVO -> B_USART1_TX
- J3 pad 2: C_VDD_BRICK -> C_SWDIO
- J3 pad 3: C_VDD_BRICK -> C_SWCLK
- J3 pad 5: C_VDD_SERVO -> C_NRST
- J3 pad 54: unconnected-(J3-Pin_54-Pad54) -> C_USART1_RX
- J3 pad 55: unconnected-(J3-Pin_55-Pad55) -> C_BRICK_VALID
- J3 pad 57: unconnected-(J3-Pin_57-Pad57) -> C_SERVO_VALID
- J3 pad 58: unconnected-(J3-Pin_58-Pad58) -> C_USB_VALID
- J3 pad 59: GND -> C_TIM4_CH4
- J3 pad 6: C_VDD_SERVO -> C_USART1_TX
- J80 pad 9: A_VDD_SERVO -> VDD_SERVO
- J81 pad 9: B_VDD_SERVO -> VDD_SERVO
- J82 pad 9: C_VDD_SERVO -> VDD_SERVO
Other:
- board text added: "ORING"

Commit message: JFOX logo as a generated KiCad silkscreen footprint
Converted from hardware/brand/jfox-logo-white.png, which is white artwork on
a transparent background - right for a presentation and wrong for a PCB in
two ways that both silently produce nothing:

  * A tracer reads DARK pixels as the shape, so white-on-transparent
    flattens to white-on-white and converts to an empty footprint.
  * The ALPHA channel carries the artwork. The RGB planes are uniform white
    wherever anything is drawn, so thresholding on brightness keeps the
    background and discards the logo.

So alpha is extracted and inverted. Not bitmap2component: KiCad ships it and
it is the obvious tool, but it is a GUI application that hangs on --help
with no console output, so it cannot be scripted.

Rectangles rather than contours. A contour tracer gives prettier polygons
and then has to solve holes, which KiCad's fp_poly has no primitive for -
and this logo is mostly holes, so every inner contour would fill in.
Rectangle decomposition handles them for free: a hole is simply an absence
of rectangles.

The generator refuses to emit art the fab cannot print. Silkscreen resolves
about 0.15 mm, so one traced pixel must be at least that. At the 8 px/mm I
tried first a pixel is 0.125 mm and 209 of 278 features came out below the
minimum - most of the logo would have arrived as broken speckle rather than
thin. It now stops with the maximum px/mm that works.

Two faults this surfaced:

  * score_fmu_layout raised "no courtyard and no pads" on the logo and took
    the whole scorer down. That guard is right for a component and wrong for
    artwork, which has neither by definition. Keying the skip off the
    board_only attribute did not work - it does not survive into the board
    file - so it keys off having no pads, which is a property of the thing
    rather than a label on it.
  * The logo lands on copper on both boards. Silkscreen over copper is
    clipped by the mask, so a logo placed there does not ap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
Parts:
- added G***: JFOX, JFOX_Logo, F.Cu at (36.0, 122.0)

Commit message: JXK-1 part numbering, from one definition
Format follows MIL-STD-130 UII Construct 2 - enterprise, part number,
serial - and the DO-254 requirement for a correlation between design data
and the as-built article.

  design identifier   JXK-1-1001-A         drawings, BOM, silkscreen
  article identifier  JXK-1-1001-A-0007    one physical unit

Part numbers are blocked so the number says what kind of thing it is:
1000s assemblies, 1100s bare boards, 1200s harnesses, 1300s mechanical,
1400s software, 1500s test equipment.

Two decisions worth recording:

  * An assembly and the bare board it is built on get DIFFERENT part
    numbers. They are different things - one is fabricated, the other
    fabricated and populated - with separate acceptance criteria. The
    SILKSCREEN carries the bare-board number, because silkscreen is applied
    before a single component is fitted and a board claiming the assembly
    number is claiming to be something it is not yet.
  * A serial is never reset when the revision changes and never reused. It
    follows the physical article for life; the revision says what standard
    that article currently conforms to. A serial that restarts per revision
    cannot support the DO-254 correlation at all.

Revision letters skip I, O, Q, S, X and Z - misread as 1, 0, 0, 5, a
cross-out and 2 on a marked board. A change that breaks interchangeability
is a new part number, not a revision; that distinction is the whole value of
the scheme.

part_numbers.py is the single definition and self-checks: block ranges,
excluded revision letters, and that no board uses one number for both its
assembly and its bare board. The schematic revision and title block, and the
board silkscreen, all import from it.

Two faults this surfaced:

  * The schematic generator OVERWROTE jfox-fmu.kicad_pro, which is where the
    PCB generator puts the net classes and design rules - KiCad rejects them
    in the board file. So the order the two happened to run in decided
    w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
Other:
- board text added: "JXK-1-1102-A"
Changed lines of the file:
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@@
 	)
+	)
+	(gr_text "JXK-1-1102-A"
+		(at 32.0 31.6)
+		(layer "F.SilkS")
+		(effects (font (size 0.8 0.8) (thickness 0.12)) (justify left))
 	)
 	(footprint "JFOX_Logo"
