File: hardware/jfox-base-v1/jfox-base.kicad_pcb (KiCad board)
At the start: 8 copper layers, 100 x 100 mm, 63 parts, among them J1 Mezz A, J100 EXP A, J101 EXP B, J102 EXP C, J2 Mezz B, J3 Mezz C, J50 PWR 1 RH, J51 PWR 2 LH, J52 DEBUG, J54 USB-C, J60 A CAN1, J61 A CAN2, J62 B CAN1, J63 B CAN2, J64 C CAN1, J65 C CAN2, J70 VEHICLE CAN, J80 ACT A, J81 ACT B, J82 ACT C, J90 GPS1 (A), J91 RC IN (B), J92 TELEM1 (A), J93 TELEM2 (C), Q1A PMOS, Q1B PMOS, Q2A PMOS, Q2B PMOS, U20 LTC4417CGN, U50 OPT1 TX, U51 OPT1 RX, U52 OPT2 TX, U53 OPT2 RX

Commit message: Provability: check the backplane, and fix the four defects that found
Nothing read JFOX-BASE-v1. Every checker in hardware/tools/ opened
jfox-fmu-v1/jfox-fmu.kicad_sch and only that, so no claim about the
backplane was provable - including the ones the requirements table recorded
as verified.

check_base_schematic.py now reads it: fused rails must reach a card socket,
the LTC4417 divider must produce the window it claims, that window must fit
every part downstream, and the feed-health outputs must reach a card AND be
driven. It failed on first run, which is the only reason to trust it.

What it found, in the order it found them:

  1. THE CARDS HAD NO POWER. The fuses put out A/B/C_FUSED and the card edge
     reads +5V_CARRIER. Both boards generated cleanly, both passed DRC, and
     the two halves were never connected to each other. The chain now
     terminates on the card rail past the shunt, not before it.

  2. THE FEEDS ARE NOT BATTERIES. VBAT_RH/VBAT_LH carry 5 V - the thresholds
     said so and the connectors are labelled PWR. Renamed PWR1_IN/PWR2_IN,
     output PWR_ORED. The name was the thing that was wrong.

  3. THE WINDOW PASSED MORE THAN A PART SURVIVES, and the binding part was
     not the one found by hand. The analysis flagged the AP2112K at 6.0 V
     against a 5.81 V threshold - 190 mV. The checker compared against every
     downstream part and found the ISOW1044 at 5.5 V: NEGATIVE 310 mV. A
     feed the controller reported as good would have destroyed the isolator.

     787k / 28k7 / 196k -> UV 4.50 V, OV 5.16 V
       ISOW1044  +338 mV      AP2112K  +838 mV

  4. THE ORING CONTROLLER'S OUTPUT WAS NEVER CONNECTED. Its pin map was
     written from the datasheet's block diagram, not the symbol: the pins
     are ~{VALID1..3} with overbars, VOUT not OUT, HYS not HYST, and there
     is no STAT pin at all. nets.get() returns None for an unknown key, so
     six pins were silently left unwired - VOUT among them. PWR_ORED was fed
     only by D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
Parts:
- R71, R74: value 49k9 -> 28k7
- R72, R75: value 174k -> 196k
Connections:
- net VBAT_LH renamed PWR2_IN
- C1 pad 1: A_VDD_BRICK -> A_+5V_CARRIER
- C2 pad 1: B_VDD_BRICK -> B_+5V_CARRIER
- C3 pad 1: C_VDD_BRICK -> C_+5V_CARRIER
- D50 pad 1: VBAT_RH -> PWR1_IN
- D50 pad 2: VBAT_IN -> PWR_ORED
- D51 pad 2: VBAT_IN -> PWR_ORED
- F1 pad 1: VBAT_IN -> PWR_ORED
- F2 pad 1: VBAT_IN -> PWR_ORED
- F3 pad 1: VBAT_IN -> PWR_ORED
- J1 pad 55: A_BRICK_VALID -> PWR1_VALID
- J1 pad 57: A_SERVO_VALID -> PWR2_VALID
- J1 pad 58: A_USB_VALID -> unconnected-(J1-Pin_58-Pad58)
- J100 pad 11: A_BRICK_VALID -> GND
- J100 pad 12: A_SERVO_VALID -> GND
- J100 pad 13: A_USB_VALID -> GND
- J2 pad 55: B_BRICK_VALID -> PWR1_VALID
- J2 pad 57: B_SERVO_VALID -> PWR2_VALID
- J2 pad 58: B_USB_VALID -> unconnected-(J2-Pin_58-Pad58)
- J3 pad 55: C_BRICK_VALID -> PWR1_VALID
- J3 pad 57: C_SERVO_VALID -> PWR2_VALID
- J3 pad 58: C_USB_VALID -> unconnected-(J3-Pin_58-Pad58)
- J50 pad 1: VBAT_RH -> PWR1_IN
- J50 pad 2: VBAT_RH -> PWR1_IN
- Q1A pad 3: VBAT_RH -> PWR1_IN
- Q1B pad 3: VBAT_IN -> PWR_ORED
- Q2B pad 3: VBAT_IN -> PWR_ORED
- R1 pad 2: A_VDD_BRICK -> A_+5V_CARRIER
- R2 pad 2: B_VDD_BRICK -> B_+5V_CARRIER
- R3 pad 2: C_VDD_BRICK -> C_+5V_CARRIER
- R70 pad 1: VBAT_RH -> PWR1_IN
- U20 pad 1: VBAT_RH -> PWR1_IN
- U20 pad 10: unconnected-(U20-~{VALID1}-Pad10) -> PWR1_VALID
- U20 pad 11: unconnected-(U20-~{VALID2}-Pad11) -> PWR2_VALID
- U20 pad 12: unconnected-(U20-~{VALID3}-Pad12) -> NC_V3
- U20 pad 15: unconnected-(U20-VOUT-Pad15) -> PWR_ORED
- U20 pad 2: unconnected-(U20-~{SHDN}-Pad2) -> PWR1_IN
- U20 pad 24: VBAT_RH -> PWR1_IN
- U20 pad 3: unconnected-(U20-HYS-Pad3) -> GND

Commit message: DO-160G protection stage, and a check that recognises parts not labels
Series inductance and an SMCJ clamp on each airframe feed, bulk on the ORed
rail, soft-start per slot. Order is deliberate - L, clamp, ORing, bulk - as
a TVS with nothing ahead of it absorbs the whole injected transient itself,
which is how a correctly chosen part still fails.

ASSUMED: section 22 pin injection LEVEL 3. It was not specified, so it is
recorded in the sheet note and in VOLTAGE_ANALYSIS.md rather than left
implicit. Level 4 or 5 need larger parts than these.

SECTION 16 POWER INTERRUPT IS NOT MET, and the arithmetic is why. Three
cards at 1.2 A riding 5.16 V down to 4.50 V need 1.8 mF for 1 ms and 364 mF
for 200 ms. 364 mF at 5 V is a supercapacitor bank. C60 is sized for the
feed-to-feed switchover the ORing stage itself creates, about 1 ms, and the
interrupt is declared not met. Meeting it means holding up at a higher
voltage ahead of the ORing or requiring the airframe to provide it - both
decisions above this board. Sizing for the case you can meet and letting the
requirement imply the other is how this goes wrong quietly.

D50/D51 retained. With the LTC4417's back-to-back pairs they are redundant
for SELECTION and cost ~0.4 V, but the pass FETs only block reverse current
in the orientation the controller drives them, and a feed connected
backwards is exactly the case where the controller has no say.

The check that verifies all this had the flaw this session keeps producing.
It tested `r.startswith("D")` - a reference designator prefix - so a board
whose clamps had been replaced by 0R resistors passed, because D60 was still
called D60. A refdes is a label someone chose; the value is what gets
fitted. It now matches against known clamp families and inductance forms,
and the negative test fails on the right line.

The inductance matcher was wrong too on first attempt: it required a
trailing H, and inductance is written 10u on a BOM, not 10uH. It rejected
every real value and repo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
Parts:
- added C60: 1800u, C_0402_1005Metric, B.Cu at (56.9, 86.5)
- added C80: 100n, C_0402_1005Metric, B.Cu at (59.2, 86.5)
- added C81: 100n, C_0402_1005Metric, B.Cu at (61.5, 86.5)
- added C82: 100n, C_0402_1005Metric, B.Cu at (56.9, 87.9)
- added D60: SMCJ6.0A, D_SMC, B.Cu at (50.0, 81.3)
- added D61: SMCJ6.0A, D_SMC, B.Cu at (107.5, 81.3)
- added R80: 10k, R_0402_1005Metric, B.Cu at (114.3, 78.5)
- added R81: 10k, R_0402_1005Metric, B.Cu at (32.9, 86.2)
- added R82: 10k, R_0402_1005Metric, B.Cu at (35.8, 86.2)
Connections:
- J50 pad 1: PWR1_IN -> PWR1_IN_RAW
- J50 pad 2: PWR1_IN -> PWR1_IN_RAW
- J51 pad 1: PWR2_IN -> PWR2_IN_RAW
- J51 pad 2: PWR2_IN -> PWR2_IN_RAW
