File: hardware/jfox-base-v1/jfox-base-oring.kicad_sch (KiCad schematic)
At the start: 13 parts, among them Q1A PMOS, Q1B PMOS, Q2A PMOS, Q2B PMOS, U20 LTC4417CGN

Commit message: Provability: check the backplane, and fix the four defects that found
Nothing read JFOX-BASE-v1. Every checker in hardware/tools/ opened
jfox-fmu-v1/jfox-fmu.kicad_sch and only that, so no claim about the
backplane was provable - including the ones the requirements table recorded
as verified.

check_base_schematic.py now reads it: fused rails must reach a card socket,
the LTC4417 divider must produce the window it claims, that window must fit
every part downstream, and the feed-health outputs must reach a card AND be
driven. It failed on first run, which is the only reason to trust it.

What it found, in the order it found them:

  1. THE CARDS HAD NO POWER. The fuses put out A/B/C_FUSED and the card edge
     reads +5V_CARRIER. Both boards generated cleanly, both passed DRC, and
     the two halves were never connected to each other. The chain now
     terminates on the card rail past the shunt, not before it.

  2. THE FEEDS ARE NOT BATTERIES. VBAT_RH/VBAT_LH carry 5 V - the thresholds
     said so and the connectors are labelled PWR. Renamed PWR1_IN/PWR2_IN,
     output PWR_ORED. The name was the thing that was wrong.

  3. THE WINDOW PASSED MORE THAN A PART SURVIVES, and the binding part was
     not the one found by hand. The analysis flagged the AP2112K at 6.0 V
     against a 5.81 V threshold - 190 mV. The checker compared against every
     downstream part and found the ISOW1044 at 5.5 V: NEGATIVE 310 mV. A
     feed the controller reported as good would have destroyed the isolator.

     787k / 28k7 / 196k -> UV 4.50 V, OV 5.16 V
       ISOW1044  +338 mV      AP2112K  +838 mV

  4. THE ORING CONTROLLER'S OUTPUT WAS NEVER CONNECTED. Its pin map was
     written from the datasheet's block diagram, not the symbol: the pins
     are ~{VALID1..3} with overbars, VOUT not OUT, HYS not HYST, and there
     is no STAT pin at all. nets.get() returns None for an unknown key, so
     six pins were silently left unwired - VOUT among them. PWR_ORED was fed
     only by D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
Parts:
- R71, R74: value 49k9 -> 28k7
- R72, R75: value 174k -> 196k
Connections:
- net VBAT_IN is gone; now on net PWR_ORED: Q1B.3 (D), Q2B.3 (D)
- net VBAT_RH is gone; now on net PWR1_IN: Q1A.3 (D), R70.1, U20.1 (EN), U20.24 (V1)
- net GND: now also U20.3 (HYS)
- net PWR1_VALID: now reaches U20.10 (~{VALID1})
- net PWR2_VALID: now reaches U20.11 (~{VALID2})
- net NC_V3: now reaches U20.12 (~{VALID3})
- net PWR_ORED: now reaches U20.15 (VOUT)
- net PWR1_IN: now reaches U20.2 (~{SHDN})
- net VBAT_LH renamed PWR2_IN
Changed lines of the file:
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@@
 		(instances
 			(project "jfox-base"
-				(path "/0eb55bbe-757b-4148-b921-b55131e0ce25"
+				(path "/c0fff4c1-c3c6-457e-a624-4248f2639ce4"
 					(reference "U20")
 					(unit 1)
@@
 		)
 	)
-	(global_label "VBAT_RH"
+	(global_label "PWR1_IN"
+		(shape bidirectional)
+		(at 73.66 90.17 0)
+		(fields_autoplaced yes)
+		(effects
+			(font
+				(size 1.27 1.27)
+			)
+			(justify left)
+		)
+	)
+	(wire
+		(pts
+			(xy 78.74 87.63) (xy 73.66 87.63)
+		)
+		(stroke
+			(width 0)
+			(type default)
+		)
+	)
+	(global_label "PWR1_IN"
+		(shape bidirectional)
+		(at 73.66 87.63 0)
+		(fields_autoplaced yes)
+		(effects
+			(font
+				(size 1.27 1.27)
+			)
+			(justify left)
+		)
+	)
+	(wire
+		(pts
+			(xy 78.74 92.71) (xy 73.66 92.71)
+		)
+		(stroke
+			(width 0)
+			(type default)
+		)
+	)
+	(global_label "GND"
 		(shape input)
-		(at 73.66 90.17 0)
+		(at 73.66 92.71 0)
 		(fields_autoplaced yes)
 		(effects
@@
 	(wire
 		(pts
+			(xy 104.14 87.63) (xy 109.22 87.63)
+		)
+		(stroke
+			(width 0)
+			(type default)
+		)
+	)
+	(global_label "PWR1_VALID"
+		(shape output)
+		(at 109.22 87.63 180)
+		(fields_autoplaced yes)
+		(effects
+			(font
+				(size 1.27 1.27)
+			)
+			(justify left)
+		)
+	)
+	(wire
+		(pts
+			(xy 104.14 90.17) (xy 109.22 90.17)
+		)
+		(stroke
+			(width 0)
+			(type default)
+		)
+	)
+	(global_label "PWR2_VALID"
+		(shape output)
+		(at 109.22 90.17 180)
+		(fields_autoplaced yes)
+		(effects
+			(font
+				(size 1.27 1.27)
+			)
+			(justify left)
+		)
+	)
+	(wire
+		(pts
+			(xy 104.14 92.71) (xy 109.22 92.71)
+		)
+		(stroke
+			(width 0)
+			(type default)
+		)
+	)
+	(global_label "NC_V3"
+		(shape bidirectional)
+		(at 109.22 92.71 180)
+		(fields_autoplaced yes)
+		(effects
+			(font
+				(size 1.27 1.27)
+			)
+			(justify left)
+		)
+	)
+	(wire
+		(pts
 			(xy 91.44 102.87) (xy 91.44 110.49)
 		)
@@
 	(wire
 		(pts
+			(xy 104.14 85.09) (xy 109.22 85.09)
+		)
+		(stroke
+			(width 0)
+			(type default)
+		)
+	)
+	(global_label "PWR_ORED"
+		(shape bidirectional)
+		(at 109.22 85.09 180)
+		(fields_autoplaced yes)
+		(effects
+			(font
+				(size 1.27 1.27)
+			)
+			(justify left)
+		)
+	)
+	(wire
+		(pts
 			(xy 104.14 77.47) (xy 109.22 77.47)
 		)
@@
 		)
 	)
-	(global_label "VBAT_LH"
-		(shape input)
+	(global_label "PWR2_IN"
+		(shape bidirectional)
 		(at 73.66 67.31 0)
 		(fields_autoplaced yes)
@@
 		)
 	)
-	(global_label "VBAT_RH"
-		(shape input)
+	(global_label "PWR1_IN"
+		(shape bidirectional)
 		(at 73.66 57.15 0)
 		(fields_autoplaced yes)
@@
 		(instances
 			(project "jfox-base"
-				(path "/0eb55bbe-757b-4148-b921-b55131e0ce25"
+				(path "/c0fff4c1-c3c6-457e-a624-4248f2639ce4"
 					(reference "Q1A")
 					(unit 1)
@@
 		)
 	)
-	(global_label "VBAT_RH"
-		(shape input)
+	(global_label "PWR1_IN"
+		(shape bidirectional)
 		(at 55.88 147.32 180)
 		(fields_autoplaced yes)
@@
 		(instances
 			(project "jfox-base"
-				(path "/0eb55bbe-757b-4148-b921-b55131e0ce25"
+				(path "/c0fff4c1-c3c6-457e-a624-4248f2639ce4"
 					(reference "Q1B")
 					(unit 1)
@@
 		)
 	)
-	(global_label "VBAT_IN"
-		(shape input)
+	(global_label "PWR_ORED"
+		(shape bidirectional)
 		(at 86.36 147.32 180)
 		(fields_autoplaced yes)
@@
 		(instances
 			(project "jfox-base"
-				(path "/0eb55bbe-757b-4148-b921-b55131e0ce25"
+				(path "/c0fff4c1-c3c6-457e-a624-4248f2639ce4"
 					(reference "Q2A")
 					(unit 1)
@@
 		)
 	)
-	(global_label "VBAT_LH"
-		(shape input)
+	(global_label "PWR2_IN"
+		(shape bidirectional)
 		(at 132.08 147.32 180)
 		(fields_autoplaced yes)
@@
 		(instances
 			(project "jfox-base"
-				(path "/0eb55bbe-757b-4148-b921-b55131e0ce25"
+				(path "/c0fff4c1-c3c6-457e-a624-4248f2639ce4"
 					(reference "Q2B")
 					(unit 1)
@@
 		)
 	)
-	(global_label "VBAT_IN"
-		(shape input)
+	(global_label "PWR_ORED"
+		(shape bidirectional)
 		(at 162.56 147.32 180)
 		(fields_autoplaced yes)
@@
 		(instances
 			(project "jfox-base"
-				(path "/0eb55bbe-757b-4148-b921-b55131e0ce25"
+				(path "/c0fff4c1-c3c6-457e-a624-4248f2639ce4"
 					(reference "R70")
 					(unit 1)
@@
 		)
 	)
-	(global_label "VBAT_RH"
+	(global_label "PWR1_IN"
 		(shape bidirectional)
 		(at 48.26 184.15 180)
@@
 		)
 		)
-		(property "Value" "49k9"
+		(property "Value" "28k7"
 			(at 72.39 203.77 0)
 			(effects
@@
 		(instances
 			(project "jfox-base"
-				(path "/0eb55bbe-757b-4148-b921-b55131e0ce25"
+				(path "/c0fff4c1-c3c6-457e-a624-4248f2639ce4"
 					(reference "R71")
 					(unit 1)
@@
 		)
 		)
-		(property "Value" "174k"
+		(property "Value" "196k"
 			(at 96.52 203.77 0)
 			(effects
@@
 		(instances
 			(project "jfox-base"
-				(path "/0eb55bbe-757b-4148-b921-b55131e0ce25"
+				(path "/c0fff4c1-c3c6-457e-a624-4248f2639ce4"
 					(reference "R72")
 					(unit 1)
@@
 		(instances
 			(project "jfox-base"
-				(path "/0eb55bbe-757b-4148-b921-b55131e0ce25"
+				(path "/c0fff4c1-c3c6-457e-a624-4248f2639ce4"
 					(reference "R73")
 					(unit 1)
@@
 		)
 	)
-	(global_label "VBAT_LH"
+	(global_label "PWR2_IN"
 		(shape bidirectional)
 		(at 120.65 184.15 180)
@@
 		)
 		)
-		(property "Value" "49k9"
+		(property "Value" "28k7"
 			(at 144.78 203.77 0)
 			(effects
@@
 		(instances
 			(project "jfox-base"
-				(path "/0eb55bbe-757b-4148-b921-b55131e0ce25"
+				(path "/c0fff4c1-c3c6-457e-a624-4248f2639ce4"
 					(reference "R74")
 					(unit 1)
@@
 		)
 		)
-		(property "Value" "174k"
+		(property "Value" "196k"
 			(at 168.91 203.77 0)
 			(effects
@@
 		(instances
 			(project "jfox-base"
-				(path "/0eb55bbe-757b-4148-b921-b55131e0ce25"
+				(path "/c0fff4c1-c3c6-457e-a624-4248f2639ce4"
 					(reference "R75")
 					(unit 1)
@@
 		(instances
 			(project "jfox-base"
-				(path "/0eb55bbe-757b-4148-b921-b55131e0ce25"
+				(path "/c0fff4c1-c3c6-457e-a624-4248f2639ce4"
 					(reference "C70")
 					(unit 1)
@@
 		(instances
 			(project "jfox-base"
-				(path "/0eb55bbe-757b-4148-b921-b55131e0ce25"
+				(path "/c0fff4c1-c3c6-457e-a624-4248f2639ce4"
 					(reference "C71")
 					(unit 1)
